File: pcb/anydice.kicad_pcb (KiCad board)
At the start: 2 copper layers, 56.6 x 48 mm, 15 parts, among them J1 Conn_01x02, SW2 SW_SPST, U1 module_mpu6050, U2 XIAO ESP32C3, U3 ER_OLEDM0.91_1x-I2C, U4 TP4056-42-ESOP8

Commit message: upd 3d files
Parts:
- moved D2 2.55 mm to (168.3, 118.5)
- moved D3 2.54 mm to (206.0, 119.5), turned to 75 degrees
Routing:
- net Net-(D2-K): track 86.5 -> 89.0 mm
- net Net-(D1-K): track 128.0 -> 130.2 mm
- net Net-(D1-A): track 46.4 -> 48.2 mm
- net GND: track 129.5 -> 130.4 mm
Other:
- outline, holes or cut-outs redrawn
